Commit message: :hammer: R2D2

File: src/basic/urdf/model.urdf (robot description, URDF)
Before this commit: robot visual, 16 links, 15 joints
Links:
- link base_link: mass None -> 10; geometry collision cylinder length=0.6 radius=0.2; visual cylinder length=0.6 radius=0.2
- link box: mass None -> 1; geometry collision box size=0.08 0.08 0.08; visual box size=0.08 0.08 0.08
- link gripper_pole: mass None -> 0.05; geometry collision cylinder length=0.2 radius=0.01; visual cylinder length=0.2 radius=0.01
- link head: mass None -> 2; geometry collision sphere radius=0.2; visual sphere radius=0.2
- link left_back_wheel: mass None -> 1; geometry collision cylinder length=0.1 radius=0.035; visual cylinder length=0.1 radius=0.035
- link left_base: mass None -> 10; geometry collision box size=0.4 0.1 0.1; visual box size=0.4 0.1 0.1
- link left_front_wheel: mass None -> 1; geometry collision cylinder length=0.1 radius=0.035; visual cylinder length=0.1 radius=0.035
- link left_gripper: mass None -> 0.05; geometry collision mesh filename=package://basic/meshes/l_finger.dae; visual mesh filename=package://basic/meshes/l_finger.dae
- link left_leg: mass None -> 10; geometry collision box size=0.6 0.1 0.2; visual box size=0.6 0.1 0.2
- link left_tip: mass None -> 0.05; geometry collision mesh filename=package://basic/meshes/l_finger_tip.dae; visual mesh filename=package://basic/meshes/l_finger_tip.dae
- link right_back_wheel: mass None -> 1; geometry collision cylinder length=0.1 radius=0.035; visual cylinder length=0.1 radius=0.035
- link right_base: mass None -> 10; geometry collision box size=0.4 0.1 0.1; visual box size=0.4 0.1 0.1
- link right_front_wheel: mass None -> 1; geometry collision cylinder length=0.1 radius=0.035; visual cylinder length=0.1 radius=0.035
- link right_gripper: mass None -> 0.05; geometry collision mesh filename=package://basic/meshes/l_finger.dae; visual mesh filename=package://basic/meshes/l_finger.dae
- link right_leg: mass None -> 10; geometry collision box size=0.6 0.1 0.2; visual box size=0.6 0.1 0.2
- link right_tip: mass None -> 0.05; geometry collision mesh filename=package://basic/meshes/l_finger_tip.dae; visual mesh filename=package://basic/meshes/l_finger_tip.dae
Joints:
- joint base_to_left_leg: origin xyz=0 0.25 0.30 -> xyz=0 0.22 0.25
- joint base_to_right_leg: origin xyz=0 -0.25 0.30 -> xyz=0 -0.22 0.25
- joint gripper_extension: limit (none) -> lower=-0.38 upper=0 effort=1000.0 velocity=0.5; type fixed -> prismatic
- joint head_swivel: axis (none) -> 0 0 1; type fixed -> continuous
- joint left_back_wheel_joint: axis (none) -> 0 1 0; type fixed -> continuous
- joint left_front_wheel_joint: axis (none) -> 0 1 0; type fixed -> continuous
- joint left_gripper_joint: axis (none) -> 0 0 1; limit (none) -> lower=0.0 upper=0.548 effort=1000.0 velocity=0.5; type fixed -> revolute
- joint right_back_wheel_joint: axis (none) -> 0 1 0; type fixed -> continuous
- joint right_front_wheel_joint: axis (none) -> 0 1 0; type fixed -> continuous
- joint right_gripper_joint: axis (none) -> 0 0 -1; limit (none) -> lower=0.0 upper=0.548 effort=1000.0 velocity=0.5; type fixed -> revolute
